File: Nordic_PCB.kicad_pcb (KiCad board)
At the start: 4 copper layers, 38.7 x 24.7 mm, 77 parts, among them J1 USB_B_Micro, J2 Conn_02x05_Counter_Clockwise, J3 Conn_01x02, J4 Conn_01x16, P1 AD5206, SW1 SW_DPDT_x2, U1 MAX9939, U2 CAP1208_QFN, U3 nrf52832, U4 DMC2400UV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

Commit message: BOM
Routing:
- net GND: track 62.5 -> 61.5 mm
Changed lines of the file:
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@@
     (thickness 1.6)
     (drawings 8)
-    (tracks 1157)
+    (tracks 1153)
     (zones 0)
     (modules 77)
@@
     (tags capacitor)
     (attr smd)
-    (fp_text reference C21 (at -2.15 0.05) (layer F.SilkS)
+    (fp_text reference C21 (at 2.065 -0.1) (layer F.SilkS)
       (effects (font (size 0.75 0.75) (thickness 0.125)))
     )
@@
   (segment (start 96.681188 106.381268) (end 96.681188 106.812603) (width 0.152) (layer F.Cu) (net 6))
   (via (at 106.00586 107.136548) (size 0.61) (drill 0.305) (layers F.Cu B.Cu) (net 6))
-  (segment (start 96.75 109.315) (end 96.75 109.02) (width 0.152) (layer F.Cu) (net 6))
   (segment (start 104.15 105.6125) (end 104.625 105.6125) (width 0.152) (layer F.Cu) (net 6))
   (via (at 96.681188 106.812603) (size 0.61) (drill 0.305) (layers F.Cu B.Cu) (net 6))
-  (segment (start 96.89587 108.87413) (end 97.452985 108.87413) (width 0.152) (layer F.Cu) (net 6))
   (segment (start 99.282456 103.78) (end 96.681188 106.381268) (width 0.152) (layer F.Cu) (net 6))
   (segment (start 104.625 105.6125) (end 106.00586 106.99336) (width 0.152) (layer F.Cu) (net 6))
-  (segment (start 96.75 109.02) (end 96.89587 108.87413) (width 0.152) (layer F.Cu) (net 6))
-  (via (at 97.452985 108.87413) (size 0.61) (drill 0.305) (layers F.Cu B.Cu) (net 6))
   (segment (start 106.00586 106.99336) (end 106.00586 107.136548) (width 0.152) (layer F.Cu) (net 6))
   (via (at 94.53 108.5) (size 0.61) (drill 0.305) (layers F.Cu B.Cu) (net 6))
@@
   (via (at 116.5 117.2) (size 0.61) (drill 0.305) (layers F.Cu B.Cu) (net 6))
   (via (at 114.4 117.2) (size 0.61) (drill 0.305) (layers F.Cu B.Cu) (net 6))
+  (via (at 97.7 108.7) (size 0.61) (drill 0.305) (layers F.Cu B.Cu) (net 6))
   (segment (start 100.715 117.685) (end 100.7 117.7) (width 0.25) (layer F.Cu) (net 7) (status 30))
   (segment (start 100.715 116.65) (end 100.715 117.685) (width 0.25) (layer F.Cu) (net 7) (status 30))
@@
   (segment (start 101.46399 100.79199) (end 100.368202 100.79199) (width 0.152) (layer B.Cu) (net 27))
   (segment (start 100.368202 100.79199) (end 100.180096 100.980096) (width 0.152) (layer B.Cu) (net 27))
-  (segment (start 91.164999 108.115001) (end 90.86 108.42) (width 0.152) (layer F.Cu) (net 27))
   (segment (start 90.87 104.580454) (end 91.018769 104.729223) (width 0.152) (layer F.Cu) (net 27))
   (segment (start 96.026023 104.086771) (end 94.964805 105.147989) (width 0.152) (layer F.Cu) (net 27))

Commit message: Design checker OK
Routing:
- net Net-(C27-Pad2): track 13.2 -> 14.2 mm
